File: DevelopmentBoards/EPS Control Unit/EPS_ControlUnit/EPS_ControlUnit.kicad_sch (KiCad schematic)
At the start: 52 parts, among them J1 Conn_01x04_Pin, J2 USB_B_Micro, J3 Conn_01x04_Pin, J4 Conn_01x04_Pin, J5 Conn_01x04_Pin, J6 Conn_01x04_Pin, J7 Conn_01x02_Pin, J8 Conn_01x04_Pin, SW1 SW_SPDT, U1 STM32L476VET6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

Commit message: Final changes to EPS Control unit dev board
Added pinouts for ADC and DAC
Sent EPS Control unit for manufacturing
Started designing EPS PDB Board (Control Unit + Power Distribution and Regulation)
Parts:
- added J10, J9: Conn_01x01_Pin, Connector_PinHeader_2.54mm:PinHeader_1x01_P2.54mm_Vertical, symbol Connector:Conn_01x01_Pin
Connections:
- net ADC: now reaches U1.15 (PC0)
- net ADC: now also J9.1 (Pin_1)
- net DAC: now reaches U1.29 (PA4)
- net DAC: now also J10.1 (Pin_1)
- no-connect marks 65 -> 63
Other:
- moved on the sheet: J8
Changed lines of the file:
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@@
   (no_connect (at 224.155 130.175))
   (no_connect (at 168.91 251.46))
-  (no_connect (at 224.155 84.455))
   (no_connect (at 224.155 94.615))
   (no_connect (at 178.435 158.115))
@@
   (no_connect (at 178.435 153.035))
   (no_connect (at 178.435 178.435))
-  (no_connect (at 224.155 160.655))
   (no_connect (at 178.435 109.855))
   (no_connect (at 224.155 112.395))
@@
     (stroke (width 0) (type default))
   )
+  (wire (pts (xy 332.74 111.76) (xy 339.725 111.76))
+    (stroke (width 0) (type default))
+  )
   (wire (pts (xy 54.61 231.775) (xy 54.61 236.22))
     (stroke (width 0) (type default))
@@
     (stroke (width 0) (type default))
   )
+  (wire (pts (xy 224.155 84.455) (xy 231.14 84.455))
+    (stroke (width 0) (type default))
+  )
   (wire (pts (xy 189.865 47.625) (xy 189.865 51.435))
     (stroke (width 0) (type default))
@@
     (stroke (width 0) (type default))
   )
-  (wire (pts (xy 336.55 105.41) (xy 343.535 105.41))
+  (wire (pts (xy 332.74 100.965) (xy 339.725 100.965))
     (stroke (width 0) (type default))
   )
@@
     (stroke (width 0) (type default))
   )
-  (wire (pts (xy 336.55 107.95) (xy 343.535 107.95))
+  (wire (pts (xy 332.74 103.505) (xy 339.725 103.505))
     (stroke (width 0) (type default))
   )
@@
     (stroke (width 0) (type default))
   )
-  (wire (pts (xy 336.55 100.33) (xy 343.535 100.33))
+  (wire (pts (xy 332.74 95.885) (xy 339.725 95.885))
     (stroke (width 0) (type default))
   )
@@
     (stroke (width 0) (type default))
   )
-  (wire (pts (xy 336.55 102.87) (xy 343.535 102.87))
+  (wire (pts (xy 332.74 98.425) (xy 339.725 98.425))
     (stroke (width 0) (type default))
   )
@@
     (stroke (width 0) (type default))
   )
+  (wire (pts (xy 332.74 115.57) (xy 339.725 115.57))
+    (stroke (width 0) (type default))
+  )
   (wire (pts (xy 163.83 51.435) (xy 163.83 53.34))
     (stroke (width 0) (type default))
@@
     (stroke (width 0) (type default))
   )
+  (wire (pts (xy 224.155 160.655) (xy 231.775 160.655))
+    (stroke (width 0) (type default))
+  )
   (wire (pts (xy 103.505 201.93) (xy 106.045 201.93))
     (stroke (width 0) (type default))
@@
     (effects (font (size 1.27 1.27)) (justify left bottom))
   )
+  (label "ADC" (at 231.775 160.655 0) (fields_autoplaced)
+    (effects (font (size 1.27 1.27)) (justify left bottom))
+  )
   (label "HSE_IN" (at 167.005 92.075 0) (fields_autoplaced)
     (effects (font (size 1.27 1.27)) (justify left bottom))
@@
     (effects (font (size 1.27 1.27)) (justify left bottom))
   )
-  (label "GPIO2" (at 343.535 102.87 0) (fields_autoplaced)
+  (label "GPIO2" (at 339.725 98.425 0) (fields_autoplaced)
     (effects (font (size 1.27 1.27)) (justify left bottom))
   )
@@
     (effects (font (size 1.27 1.27)) (justify left bottom))
   )
-  (label "GPIO1" (at 343.535 100.33 0) (fields_autoplaced)
+  (label "GPIO1" (at 339.725 95.885 0) (fields_autoplaced)
     (effects (font (size 1.27 1.27)) (justify left bottom))
   )
@@
     (effects (font (size 1.27 1.27)) (justify left bottom))
   )
-  (label "GPIO4" (at 343.535 107.95 0) (fields_autoplaced)
+  (label "GPIO4" (at 339.725 103.505 0) (fields_autoplaced)
     (effects (font (size 1.27 1.27)) (justify left bottom))
   )
@@
     (effects (font (size 1.27 1.27)) (justify left bottom))
   )
+  (label "DAC" (at 231.14 84.455 0) (fields_autoplaced)
+    (effects (font (size 1.27 1.27)) (justify left bottom))
+  )
   (label "USB_D-" (at 231.14 102.235 0) (fields_autoplaced)
     (effects (font (size 1.27 1.27)) (justify left bottom))
@@
     (effects (font (size 1.27 1.27)) (justify left bottom))
   )
-  (label "GPIO3" (at 343.535 105.41 0) (fields_autoplaced)
+  (label "GPIO3" (at 339.725 100.965 0) (fields_autoplaced)
     (effects (font (size 1.27 1.27)) (justify left bottom))
   )
@@
     (effects (font (size 1.27 1.27)) (justify left bottom))
   )
+  (label "DAC" (at 339.725 115.57 0) (fields_autoplaced)
+    (effects (font (size 1.27 1.27)) (justify left bottom))
+  )
   (label "NRST" (at 258.445 256.54 0) (fields_autoplaced)
     (effects (font (size 1.27 1.27)) (justify left bottom))
@@
     (effects (font (size 1.27 1.27)) (justify left bottom))
   )
+  (label "ADC" (at 339.725 111.76 0) (fields_autoplaced)
+    (effects (font (size 1.27 1.27)) (justify left bottom))
+  )
   (label "GPIO3" (at 168.275 122.555 0) (fields_autoplaced)
     (effects (font (size 1.27 1.27)) (justify left bottom))
@@
     )
   )
+  (symbol (lib_id "Connector:Conn_01x01_Pin") (at 327.66 111.76 0) (unit 1)
+    (in_bom yes) (on_board yes) (dnp no)
+    (property "Reference" "J9" (at 325.12 106.68 0)
+      (effects (font (size 1.27 1.27)))
+    )
+    (property "Value" "Conn_01x01_Pin" (at 327.025 108.585 0)
+      (effects (font (size 1.27 1.27)))
+    )
+    (property "Footprint" "Connector_PinHeader_2.54mm:PinHeader_1x01_P2.54mm_Vertical" (at 327.66 111.76 0)
+      (effects (font (size 1.27 1.27)) hide)
+    )
+    (property "Datasheet" "~" (at 327.66 111.76 0)
+      (effects (font (size 1.27 1.27)) hide)
+    )
+    (pin "1")
+    (instances
+      (project "EPS_ControlUnit"
+        (path "/b7b561f9-f781-4e48-9d8e-6eb1511b4888"
+          (reference "J9") (unit 1)
+        )
+      )
+    )
+  )
   (symbol (lib_id "power:GND") (at 77.47 213.995 0) (unit 1)
     (in_bom yes) (on_board yes) (dnp no) (fields_autoplaced)
@@
     )
   )
-  (symbol (lib_id "Connector:Conn_01x04_Pin") (at 331.47 102.87 0) (unit 1)
+  (symbol (lib_id "Connector:Conn_01x04_Pin") (at 327.66 98.425 0) (unit 1)
     (in_bom yes) (on_board yes) (dnp no)
-    (property "Reference" "J8" (at 329.565 104.775 0)
+    (property "Reference" "J8" (at 325.755 100.33 0)
       (effects (font (size 1.27 1.27)) (justify right))
     )
-    (property "Value" "Conn_01x04_Pin" (at 334.645 96.52 0)
+    (property "Value" "Conn_01x04_Pin" (at 330.835 92.075 0)
       (effects (font (size 1.27 1.27)) (justify right))
     )
-    (property "Footprint" "Connector_PinHeader_2.54mm:PinHeader_1x04_P2.54mm_Vertical" (at 331.47 102.87 0)
+    (property "Footprint" "Connector_PinHeader_2.54mm:PinHeader_1x04_P2.54mm_Vertical" (at 327.66 98.425 0)
       (effects (font (size 1.27 1.27)) hide)
     )
-    (property "Datasheet" "~" (at 331.47 102.87 0)
+    (property "Datasheet" "~" (at 327.66 98.425 0)
       (effects (font (size 1.27 1.27)) hide)
     )
@@
         )
       )
+    )
+  )
+  (symbol (lib_id "Connector:Conn_01x01_Pin") (at 327.66 115.57 0) (unit 1)
+    (in_bom yes) (on_board yes) (dnp no)
+    (property "Reference" "J10" (at 323.85 116.84 0)
+      (effects (font (size 1.27 1.27)))
+    )
+    (property "Value" "Conn_01x01_Pin" (at 327.025 118.745 0)
+      (effects (font (size 1.27 1.27)))
+    )
+    (property "Footprint" "Connector_PinHeader_2.54mm:PinHeader_1x01_P2.54mm_Vertical" (at 327.66 115.57 0)
+      (effects (font (size 1.27 1.27)) hide)
+    )
+    (property "Datasheet" "~" (at 327.66 115.57 0)
+      (effects (font (size 1.27 1.27)) hide)
+    )
+    (pin "1")
+    (instances
+      (project "EPS_ControlUnit"
+        (path "/b7b561f9-f781-4e48-9d8e-6eb1511b4888"
+          (reference "J10") (unit 1)
+        )
+      )
