File: EPS Board/EPS_PDB/EPS_PDB.kicad_sch (KiCad schematic)
At the start: 20 parts, among them J1 USB_B_Micro, J2 Conn_02x26_Odd_Even, J3 Conn_02x26_Odd_Even, J4 Conn_01x04_Pin, U1 AMS1117-3.3

Commit message: Progresss in EPS PDB Layout
Voltage Converters and Current limiter section pending
Might need to increase trace width of power traces on inner layers
Parts:
- removed TP1: TestPoint, TestPoint:TestPoint_Pad_D2.0mm, symbol Connector:TestPoint
- removed TP2: TestPoint, TestPoint:TestPoint_Pad_2.0x2.0mm, symbol Connector:TestPoint
Changed lines of the file:
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@@
 	)
 	(junction
-		(at 238.76 254)
-		(diameter 0)
-		(color 0 0 0 0)
-	)
-	(junction
 		(at 243.205 234.315)
 		(diameter 0)
@@
 	)
 	(junction
-		(at 216.535 228.6)
-		(diameter 0)
-		(color 0 0 0 0)
-	)
-	(junction
 		(at 216.535 234.315)
 		(diameter 0)
@@
 	(wire
 		(pts
-			(xy 238.76 254) (xy 238.76 258.445)
-		)
-		(stroke
-			(width 0)
-			(type default)
-		)
-	)
-	(wire
-		(pts
 			(xy 36.83 145.415) (xy 55.245 145.415)
 		)
@@
 	(wire
 		(pts
-			(xy 216.535 225.425) (xy 216.535 228.6)
-		)
-		(stroke
-			(width 0)
-			(type default)
-		)
-	)
-	(wire
-		(pts
 			(xy 318.135 202.565) (xy 329.565 202.565)
 		)
@@
 	(wire
 		(pts
-			(xy 261.62 254) (xy 238.76 254)
-		)
-		(stroke
-			(width 0)
-			(type default)
-		)
-	)
-	(wire
-		(pts
 			(xy 314.96 116.84) (xy 321.31 116.84)
 		)
@@
 	(wire
 		(pts
-			(xy 238.76 254) (xy 216.535 254)
+			(xy 216.535 254) (xy 261.62 254)
 		)
 		(stroke
@@
 	(wire
 		(pts
-			(xy 240.665 258.445) (xy 238.76 258.445)
-		)
-		(stroke
-			(width 0)
-			(type default)
-		)
-	)
-	(wire
-		(pts
 			(xy 314.96 152.4) (xy 325.12 152.4)
 		)
@@
 	)
 	(symbol
-		(lib_id "Connector:TestPoint")
-		(at 216.535 225.425 0)
-		(mirror y)
-		(unit 1)
-		(exclude_from_sim no)
-		(in_bom yes)
-		(on_board yes)
-		(dnp no)
-		(property "Reference" "TP1"
-			(at 213.995 221.488 0)
-			(effects
-				(font
-					(size 1.27 1.27)
-				)
-				(justify left)
-			)
-		)
-		(property "Value" "TestPoint"
-			(at 213.995 224.028 0)
-			(effects
-				(font
-					(size 1.27 1.27)
-				)
-				(justify left)
-			)
-		)
-		(property "Footprint" "TestPoint:TestPoint_Pad_D2.0mm"
-			(at 211.455 225.425 0)
-			(effects
-				(font
-					(size 1.27 1.27)
-				)
-				(hide yes)
-			)
-		)
-		(property "Datasheet" "~"
-			(at 211.455 225.425 0)
-			(effects
-				(font
-					(size 1.27 1.27)
-				)
-				(hide yes)
-			)
-		)
-		(property "Description" ""
-			(at 216.535 225.425 0)
-			(effects
-				(font
-					(size 1.27 1.27)
-				)
-				(hide yes)
-			)
-		)
-		(pin "1"
-		)
-		(instances
-			(project "EPS_PDB"
-				(path "/b6081578-ab04-44e2-a71a-4911a5b750e4"
-					(reference "TP1")
-					(unit 1)
-				)
-			)
-			(project "EPS_ControlUnit"
-				(path "/b7b561f9-f781-4e48-9d8e-6eb1511b4888"
-					(reference "TP3")
-					(unit 1)
-				)
-			)
-		)
-	)
-	(symbol
 		(lib_id "Connector_Generic:Conn_02x26_Odd_Even")
 		(at 307.34 144.78 0)
@@
 					(unit 1)
 				)
-			)
-		)
-	)
-	(symbol
-		(lib_id "Connector:TestPoint")
-		(at 240.665 258.445 270)
-		(mirror x)
-		(unit 1)
-		(exclude_from_sim no)
-		(in_bom yes)
-		(on_board yes)
-		(dnp no)
-		(property "Reference" "TP2"
-			(at 245.11 256.54 90)
-			(effects
-				(font
-					(size 1.27 1.27)
-				)
-				(justify left)
-			)
-		)
-		(property "Value" "TestPoint"
-			(at 245.11 259.08 90)
-			(effects
-				(font
-					(size 1.27 1.27)
-				)
-				(justify left)
-			)
-		)
-		(property "Footprint" "TestPoint:TestPoint_Pad_2.0x2.0mm"
-			(at 240.665 253.365 0)
-			(effects
-				(font
-					(size 1.27 1.27)
-				)
-				(hide yes)
-			)
-		)
-		(property "Datasheet" "~"
-			(at 240.665 253.365 0)
-			(effects
-				(font
-					(size 1.27 1.27)
-				)
-				(hide yes)
-			)
-		)
-		(property "Description" ""
-			(at 240.665 258.445 0)
-			(effects
-				(font
-					(size 1.27 1.27)
-				)
-				(hide yes)
-			)
-		)
-		(pin "1"
-		)
-		(instances
-			(project "EPS_PDB"
-				(path "/b6081578-ab04-44e2-a71a-4911a5b750e4"
-					(reference "TP2")
-					(unit 1)
-				)
-			)
-			(project "EPS_ControlUnit"
-				(path "/b7b561f9-f781-4e48-9d8e-6eb1511b4888"
-					(reference "TP4")
-					(unit 1)
-				)
