File: EPS Board/EPS_PDB/EPS_PDB.kicad_pcb (KiCad board)
At the start: 4 copper layers, 92 x 92 mm, 126 parts, among them J1 USB_B_Micro, J2 Conn_02x26_Odd_Even, J3 Conn_02x26_Odd_Even, J4 Conn_01x04_Pin, Q1 PMOS, Q2 PMOS, SW1 SW_SPDT, U1 AMS1117-3.3, U10 TPS259621DDAT_5V_PAY, U11 LM5000-3MTCX, U12 TPS259621DDAT_5V_EPS, U13 TPS259621DDAT_5V_OBC, U14 AD7708BRUZ, U15 TPS259621DDAT_5V_ADCS, U16 TPS259621DDAT_5V_COMM, U17 LTC3624EMSE-3.3PBF, U18 TPS259621DDAT_12V_ADCS, U19 LTC3624IDD-25PBF, U2 SN65HVD256D, U3 SN65HVD256D, U4 STM32L476VET6, U5 TPS3824-33QDBVRQ1, U6 TS4061BICT-1.25, U7 TPS259621DDAT 3V3_ADCS, U8 TPS259621DDAT_3V3_ANT, U9 TPS259621DDAT_3V3_EPS, Y1 32MHz, Y2 32.768kHz

Commit message: minor layout commit
Parts:
- added C38: 4.7uF, Capacitor_SMD:C_0603_1608Metric, F.Cu at (92.8, 118.1)
- added C39: 4.7uF, Capacitor_SMD:C_0603_1608Metric, F.Cu at (92.8, 120.6)
- added C40: 1uF, Capacitor_SMD:C_0603_1608Metric, F.Cu at (146.8, 100.7)
- added C41: 1uF, Capacitor_SMD:C_0603_1608Metric, F.Cu at (126.1, 100.4)
- added C42: 1uF, Capacitor_SMD:C_0603_1608Metric, F.Cu at (136.4, 100.6)
- added C43: 1uF, Capacitor_SMD:C_0603_1608Metric, F.Cu at (157.7, 100.4)
- added C44: 1uF, Capacitor_SMD:C_0603_1608Metric, F.Cu at (168.0, 100.1)
- added C45: 1uF, Capacitor_SMD:C_0603_1608Metric, F.Cu at (176.7, 96.4)
- added C46: 1uF, Capacitor_SMD:C_0603_1608Metric, F.Cu at (197.6, 90.1)
- added C47: 1uF, Capacitor_SMD:C_0603_1608Metric, F.Cu at (186.3, 97.1)
- added C48: 1uF, Capacitor_SMD:C_0603_1608Metric, F.Cu at (197.2, 113.2)
- added D6: D_Schottky, Diode_SMD:D_0805_2012Metric, F.Cu at (169.6, 107.7)
- C20: value 10uF -> 0.1uF
- C21: value 10uF -> 100pF
- C22: value TBD -> 3300pF
- C23: value TBD -> 10nF
- C24: value TBD -> 4.7uF
- C30: value 4.7uF -> 47uF
- L1: value 16uH -> 8.2uH
- L2: value 16uH -> 2uH
- L3: value 1.3uH -> 0.9uH
- R30: value TBD -> 18k
- moved D3 100.1 mm to (174.2, 48.6)
- moved R13 43.2 mm to (147.0, 105.3), turned to -90 degrees
- moved R16 21.8 mm to (98.0, 120.5), turned to 180 degrees
- moved R14 15.0 mm to (126.3, 105.0), turned to -90 degrees
- moved R15 11.7 mm to (136.8, 105.3), turned to -90 degrees
- moved R17 10.5 mm to (103.2, 113.5)
- moved R19 10.5 mm to (102.5, 121.8)
- moved R20 10.5 mm to (102.2, 118.0)
- moved R23 10.5 mm to (97.2, 126.5)
- moved R24 10.5 mm to (98.3, 115.5)
- moved C30 4.83 mm to (130.9, 112.7)
- moved L2 2.40 mm to (125.0, 118.9)
- moved U17 2.21 mm to (133.2, 118.7)
Connections:
- net /EPS Power Distribution/MODE renamed Net-(JP3-C)
- C34 pad 1: /VBUS -> GND
- C34 pad 2: Net-(U17-RUN) -> /VBUS
- C36 pad 1: /VBUS -> GND
- C36 pad 2: Net-(U19-RUN) -> /VBUS
- JP5 pad 2: Net-(JP5-B) -> Net-(JP5-C)
- U17 pad 3: Net-(U17-RUN) -> /VBUS
- U17 pad 4: Net-(U17-RUN) -> /VBUS
- U17 pad 5: Net-(U17-RUN) -> /VBUS
- U19 pad 2: Net-(U19-RUN) -> /VBUS
- U19 pad 3: Net-(U19-RUN) -> /VBUS
- U19 pad 7: Net-(JP5-B) -> Net-(JP5-C)
Routing:
- net GND: track 92.3 -> 106.2 mm, vias 48 -> 60
- net Net-(U12-OVCSEL): track 0.00 -> 4.44 mm
- net 5V_EPS: track 142.6 -> 146.5 mm
- net Net-(U13-OVCSEL): track 0.00 -> 3.75 mm
- net Net-(U16-OVCSEL): track 0.00 -> 3.34 mm
- net /FLT_3V3_ANT: track 65.6 -> 63.1 mm, vias 5 -> 4
- net /12V_ADCS: track 86.4 -> 88.2 mm
- net 3V3_EPS: track 451.4 -> 453.1 mm
- net /3V3_ADCS: track 79.7 -> 81.4 mm
- net /3V3_ANT: track 53.4 -> 55.1 mm
- net /FLT_3V3_ADCS: track 49.5 -> 47.8 mm
- net /5V_PAY: track 54.2 -> 55.9 mm
- net /FLT_5V_COMM: track 27.4 -> 28.9 mm
- net VUSB: track 30.2 -> 31.6 mm
- net /EN_12V_ADCS: track 56.7 -> 58.0 mm
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
Commit message: EPS PDB Board LTC36424 3V3 Layout done
Parts:
- removed C40, C41, C42, C43, C44, C45, C46, C47, C48: 1uF, Capacitor_SMD:C_0603_1608Metric
- added C49: 1uF, Capacitor_SMD:C_0603_1608Metric, F.Cu at (126.1, 100.5)
- added C50: 1uF, Capacitor_SMD:C_0603_1608Metric, F.Cu at (146.8, 100.9)
- added C51: 1uF, Capacitor_SMD:C_0603_1608Metric, F.Cu at (136.5, 100.7)
- added C52: 1uF, Capacitor_SMD:C_0603_1608Metric, F.Cu at (92.6, 147.6)
- added C53: 1uF, Capacitor_SMD:C_0603_1608Metric, F.Cu at (92.6, 150.1)
- added C54: 1uF, Capacitor_SMD:C_0603_1608Metric, F.Cu at (96.7, 140.1)
- added C55: 1uF, Capacitor_SMD:C_0603_1608Metric, F.Cu at (96.7, 142.6)
- added C56: 1uF, Capacitor_SMD:C_0603_1608Metric, F.Cu at (96.7, 145.1)
- added C_12V1: 1uF, Capacitor_SMD:C_1206_3216Metric, F.Cu at (134.1, 152.5)
- added R42: 10k, Resistor_SMD:R_0603_1608Metric, F.Cu at (173.1, 112.3)
- added R43: 10k, Resistor_SMD:R_0603_1608Metric, F.Cu at (147.3, 110.8)
- C24_12V1: renamed from C24; footprint Capacitor_SMD:C_0603_1608Metric -> Capacitor_SMD:C_1206_3216Metric
- C30, C34, C35, C36: footprint Capacitor_SMD:C_0603_1608Metric -> Capacitor_SMD:C_1206_3216Metric
- C39_12V1: renamed from C39; footprint Capacitor_SMD:C_0603_1608Metric -> Capacitor_SMD:C_1206_3216Metric
- D4: footprint Diode_SMD:D_0805_2012Metric -> Diode_SMD:D_1206_3216Metric
- L2: value 2uH -> 2.2uH; footprint Inductor-WE-XHMI-5050:WE-XHMI-5050 -> Inductor_SMD:L_Wuerth_WE-XHMI-8080
- L3: value 0.9uH -> 2.2uH; footprint Inductor_SMD:L_1206_3216Metric -> Inductor_SMD:L_Wuerth_WE-XHMI-8080
- moved C39_12V1 72.2 mm to (159.9, 147.1)
- moved JP5 20.5 mm to (166.4, 115.4), turned to 180 degrees
- moved JP3 16.8 mm to (138.2, 114.4), turned to 180 degrees
- moved C37 11.8 mm to (162.7, 115.0), turned to -90 degrees
- moved C33 11.6 mm to (133.9, 114.7), turned to -90 degrees
- moved L1 7.25 mm to (174.6, 122.9)
- moved L3 6.55 mm to (154.9, 118.2), turned to -90 degrees
- moved U19 6.34 mm to (162.4, 118.6)
- moved C35 5.24 mm to (160.1, 112.0)
- moved C20 4.16 mm to (175.8, 127.7)
- moved C21 4.11 mm to (179.4, 117.5)
- moved C36 3.96 mm to (164.5, 122.0), turned to 180 degrees
- moved C19 2.78 mm to (178.9, 130.0)
- moved R25 2.78 mm to (192.8, 129.6)
- moved R30 2.78 mm to (188.2, 132.5)
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Connections:
- net Net-(JP3-B) renamed /EPS Power Distribution/INTVCC_3V3
- net Net-(JP3-C) renamed /EPS Power Distribution/MODE_3V3
- net Net-(L2-Pad2) renamed /EPS Power Distribution/SW_3V3
- net Net-(U19-SW) renamed /EPS Power Distribution/SW_5V
- C19 pad 2: /EPS Power Distribution/VIN -> /VBUS
- C35 pad 1: /EPS Power Distribution/5V_BUS -> GND
- C35 pad 2: GND -> /EPS Power Distribution/5V_BUS
- R25 pad 1: /EPS Power Distribution/VIN -> /VBUS
- U11 pad 13: /EPS Power Distribution/VIN -> /VBUS
Routing:
- net /STATUS_3V3: track 0.00 -> 87.8 mm, vias 0 -> 9
- net /FLT_3V3_ANT: track 63.1 -> 72.9 mm, vias 4 -> 5
- net /EPS Power Distribution/MODE_3V3: track 0.00 -> 9.25 mm
- net /EPS Power Distribution/3.3V_BUS: track 0.00 -> 7.85 mm, vias 0 -> 2
- net /EPS Power Distribution/INTVCC_3V3: track 0.00 -> 5.29 mm
- net /EN_3V3_ANT: track 86.0 -> 83.0 mm, vias 4 -> 5
- net GND: track 106.2 -> 107.7 mm, vias 60 -> 80
- added copper zone on F.Cu, net /EPS Power Distribution/3.3V_BUS
- added copper zone on F.Cu, net /EPS Power Distribution/SW_3V3
- added copper zone on F.Cu, net /EPS Power Distribution/SW_5V
- added copper zone on F.Cu, net /VBUS

Commit message: EPS PDB Layout almost complete
Silkscreen and some minor DRC Issues to be sorted
Parts:
- removed the R14 at (126.3, 105.0)
- added R15: 10k, Resistor_SMD:R_0603_1608Metric, F.Cu at (126.3, 105.2)
- C24: renamed from C20; moved to B.Cu
- C28: renamed from C23; moved to B.Cu
- C45: renamed from C_12V1; footprint Capacitor_SMD:C_1206_3216Metric -> Capacitor_SMD:C_0603_1608Metric
- D5: renamed from D6; moved to B.Cu
- R23: renamed from R20; moved to B.Cu
- R3: renamed from R2; value R -> 100k
- R4: renamed from R3; value R -> 100
- R6: renamed from R5; value R -> 100k
- R7: renamed from R6; value R -> 100
- moved C42 113.7 mm to (197.6, 90.2)
- moved C43 101.7 mm to (186.3, 97.1)
- moved R25 100.2 mm to (198.3, 109.9)
- moved R24 93.6 mm to (185.5, 95.5)
- moved C33 91.9 mm to (167.2, 96.4)
- moved C34 91.4 mm to (176.9, 96.3)
- moved C22 88.4 mm to (180.2, 131.0), turned to 180 degrees
- moved R23 86.9 mm to (184.6, 90.5), turned to -90 degrees
- moved C26 80.3 mm to (157.7, 100.6), turned to -90 degrees
- moved R22 78.3 mm to (174.2, 90.2), turned to 180 degrees
- moved C45 74.3 mm to (197.2, 113.3), turned to -90 degrees
- moved R20 67.5 mm to (169.1, 99.1)
- moved R19 62.3 mm to (155.7, 97.1), turned to 0 degrees
- moved C31 41.0 mm to (193.5, 123.6), turned to -90 degrees
- moved R41 39.0 mm to (137.2, 97.0), turned to 180 degrees
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- renumbered C50 to C17, C49 to C18, C17 to C19, C18 to C20, C51 to C21, C38 to C22, C19 to C23, C21 to C25, C52 to C26, C22 to C27, C25 to C29, C26 to C30, C39_12V1 to C31, C24_12V1 to C32, C53 to C33, C54 to C34, C27 to C35, C28 to C36, C29 to C37, C31 to C38, C32 to C39, C30 to C40, C33 to C41, C55 to C42, C56 to C43, C34 to C44, C37 to C46, C35 to C47, C36 to C48, D5 to D1, D1 to D2, D2 to D3, D3 to D4, D4 to D6, J4 to J2, J2 to J3, J3 to J4, JP6 to JP1, JP1 to JP3, JP3 to JP4, JP4 to JP5, JP5 to JP6, R41 to R1, R9 to R10, R10 to R11, R11 to R12, R12 to R13, R13 to R14, R15 to R16, R21 to R17, R22 to R18, R16 to R19, R1 to R2, R17 to R20, R18 to R21, R19 to R22, R23 to R24, R24 to R25, R27 to R26, R25 to R27, R29 to R28, R30 to R29, R31 to R30, R26 to R31, R28 to R32, R32 to R33, R33 to R34, R34 to R35, R35 to R36, R36 to R37, R37 to R38, R38 to R39, R39 to R40, R42 to R41, R43 to R42, R40 to R43, R4 to R5, R7 to R9, U17 to U15, U15 to U16, U16 to U17, U7 to U6, U8 to U7, U6 to U8
Connections:
- net Net-(D4-A) renamed /EPS Power Distribution/SW_12V
- net Net-(JP5-B) renamed /EPS Power Distribution/INTVCC_5V
- net Net-(JP5-C) renamed /EPS Power Distribution/MODE_5V
- C23 pad 2: /VBUS -> /EPS Power Distribution/VIN_12V
- C27 pad 1: Net-(C22-Pad1) -> GND
- C27 pad 2: Net-(U11-COMP) -> Net-(C27-Pad2)
- C31 pad 1: GND -> /EPS Power Distribution/12V_BUS
- C31 pad 2: /EPS Power Distribution/12V_BUS -> GND
- C32 pad 1: GND -> /EPS Power Distribution/12V_BUS
- C32 pad 2: /EPS Power Distribution/12V_BUS -> GND
- J1 pad 6: unconnected-(J1-Shield-Pad6)_5 -> GND
- R14 pad 2: /EPS Power Distribution/3.3V_BUS -> 3V3_EPS
- R19 pad 2: /EPS Power Distribution/3.3V_BUS -> 3V3_EPS
- R20 pad 2: /EPS Power Distribution/3.3V_BUS -> 3V3_EPS
- R22 pad 2: /EPS Power Distribution/3.3V_BUS -> 3V3_EPS
- R23 pad 2: /EPS Power Distribution/3.3V_BUS -> 3V3_EPS
- R24 pad 2: /EPS Power Distribution/3.3V_BUS -> 3V3_EPS
- R25 pad 2: /EPS Power Distribution/3.3V_BUS -> 3V3_EPS
- R27 pad 1: /VBUS -> /EPS Power Distribution/VIN_12V
- R28 pad 2: /EPS Power Distribution/12V -> /EPS Power Distribution/FB_12V
- R29 pad 1: Net-(C22-Pad1) -> Net-(U11-COMP)
- R29 pad 2: GND -> Net-(C27-Pad2)
- R30 pad 1: GND -> /EPS Power Distribution/FB_12V
- R30 pad 2: /EPS Power Distribution/12V -> GND
- R41 pad 2: /EPS Power Distribution/3.3V_BUS -> 3V3_EPS
- U11 pad 13: /VBUS -> /EPS Power Distribution/VIN_12V
- U11 pad 2: /EPS Power Distribution/12V -> /EPS Power Distribution/FB_12V
Routing:
- net /STATUS_5V: track 0.00 -> 91.2 mm, vias 0 -> 4
- net /SHDN_12V: track 0.00 -> 74.6 mm, vias 0 -> 4
- net 3V3_EPS: track 453.1 -> 498.4 mm, vias 12 -> 19
- net GND: track 107.7 -> 144.5 mm, vias 80 -> 128
- net /EPS Control Unit/CAN_SW_B: track 33.9 -> 53.0 mm, vias 4 -> 6
- net /FLT_3V3_EPS: track 44.7 -> 54.6 mm, vias 4 -> 5
- net /EPS Power Distribution/5V_BUS: track 0.00 -> 8.80 mm, vias 0 -> 2
- net /EPS Power Distribution/MODE_5V: track 0.00 -> 7.73 mm
- net /EPS Power Distribution/VIN_12V: track 0.00 -> 6.19 mm
- net /EPS Power Distribution/12V_BUS: track 0.00 -> 4.41 mm
- net /EPS Power Distribution/INTVCC_5V: track 0.00 -> 3.96 mm
- net /FLT_5V_EPS: track 49.1 -> 52.8 mm, vias 2 -> 3
- net /EPS Power Distribution/FB_12V: track 0.00 -> 3.71 mm
- net Net-(U16-OVCSEL): track 0.00 -> 3.67 mm
- net /5V_ADCS: track 25.6 -> 29.1 mm
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- added copper zone on In1.Cu, net /5V_ADCS
- added copper zone on F.Cu, net /EPS Power Distribution/12V_BUS
- added copper zone on F.Cu, net /EPS Power Distribution/5V_BUS
- added copper zone on F.Cu, net /EPS Power Distribution/SW_12V
- added copper zone on In1.Cu, net /VBUS

Commit message: EPS PDB Layout Complete
Have ordered the board
Parts:
- added G***: LOGO, IITBSSP Logo:IITBSSP_Logo, B.Cu at (136.0, 111.7)
- renumbered D1 to 3V3_LED, D2 to 5V_LED, D3 to HEARTBEAT
Routing:
- net VUSB: track 31.6 -> 32.5 mm
- net GND: vias 128 -> 126
- net /VBUS: vias 23 -> 12
Other:
- board text added: "12V"
- board text added: "3V3"
- board text added: "3V3_EPS"
- board text added: "5V"
- board text added: "5VUSB_POW"
- board text added: "ADCS 3V3"
- board text added: "ADCS 5V"
- board text added: "ANT"
- board text added: "COMM 5V"
- board text added: "DEBUG"
- board text added: "EPS 5V"
- board text added: "EPS POWER DISTRIBUTION BOARD AMEYA MARAKARKANDY"
- board text added: "EPS POWER DISTRIBUTION BOARD AMEYA MARAKARKANDY REV1.0 OCT 2024"
- board text added: "GND"
- board text added: "LDO EN"
- board text added: "MADE BY HUMANS FROM EARTH"
- board text added: "OBC 5V"
- board text added: "PAY 5V"
- board text added: "REV 1.0 OCT 24"
- board text added: "SCLK"
- board text added: "SWDIO"
- board text added: "VBUS CONN"
- board text removed: "EPS POWER DISTRIBUTION BOARD"
