File: EPS Board/EPS_PDB/EPS_ControlUnit.kicad_sch (KiCad schematic)
At the start: 35 parts, among them Q1 PMOS, Q2 PMOS, SW1 SW_SPDT, U2 SN65HVD256D, U3 SN65HVD256D, U4 STM32L476VET6, U5 TPS3824-33QDBVRQ1, Y1 32MHz

Commit message: EPS PDB Layout
Power Distribution and Regulation unit layout started
Parts:
- SW1: footprint Button_Switch_SMD:SW_SPST_B3S-1100 -> Button_Switch_SMD:SW_SPST_B3U-1100P
Connections:
- net PMOS1_GATE: now reaches Q1.2 (G), R2.1, R3.2
- net PMOS2_GATE: now reaches Q2.2 (G), R5.1, R6.2
Changed lines of the file:
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@@
+		)
+	)
+	(label "PMOS2_GATE"
+		(at 288.29 98.425 0)
+		(fields_autoplaced yes)
+		(effects
+			(font
+				(size 1 1)
+			)
+			(justify left bottom)
 		)
 	)
@@
 			)
 			(justify right bottom)
+		)
+	)
+	(label "PMOS1_GATE"
+		(at 287.02 68.58 0)
+		(fields_autoplaced yes)
+		(effects
+			(font
+				(size 1 1)
+			)
+			(justify left bottom)
 		)
 	)
@@
 			)
 		)
-		(property "Footprint" "Button_Switch_SMD:SW_SPST_B3S-1100"
+		(property "Footprint" "Button_Switch_SMD:SW_SPST_B3U-1100P"
 			(at 59.69 88.265 0)
 			(effects

Commit message: Progresss in EPS PDB Layout
Voltage Converters and Current limiter section pending
Might need to increase trace width of power traces on inner layers
Connections:
- net RESET_ADC: now also U4.77 (PA15)
- no-connect marks 34 -> 33
Changed lines of the file:
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@@
 	)
 	(no_connect
-		(at 140.97 121.285)
-	)
-	(no_connect
 		(at 140.97 194.945)
 	)
@@
 	(wire
 		(pts
+			(xy 140.97 121.285) (xy 153.67 121.285)
+		)
+		(stroke
+			(width 0)
+			(type default)
+		)
+	)
+	(wire
+		(pts
 			(xy 63.5 115.57) (xy 63.5 125.095)
 		)
@@
 		(fields_autoplaced yes)
 		(effects
+			(font
+				(size 1.27 1.27)
+			)
+			(justify right bottom)
+		)
+	)
+	(label "RESET_ADC"
+		(at 153.67 121.285 180)
+		(fields_autoplaced yes)
+		(effects

Commit message: EPS PDB Layout almost complete
Silkscreen and some minor DRC Issues to be sorted
Parts:
- R3: renamed from R2; value R -> 100k
- R4: renamed from R3; value R -> 100
- R6: renamed from R5; value R -> 100k
- R7: renamed from R6; value R -> 100
- renumbered D2 to D3, R9 to R10, R10 to R11, R11 to R12, R12 to R13, R4 to R5, R7 to R9

Commit message: minor changes
Other:
- note removed: "GPIO PINS ASSIGNMENT (x18) IN PROGRESS"
- note removed: "IN PROGRESS"
- note removed: "RESISTOR SIZING"
Changed lines of the file:
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@@
 	(wire
 		(pts
-			(xy 163.195 72.39) (xy 163.195 76.2)
+			(xy 163.195 72.39) (xy 163.195 75.565)
 		)
 		(stroke
@@
 	(text "Switching between\nCAN_A and CAN_B"
 		(exclude_from_sim no)
-		(at 245.11 46.355 0)
+		(at 254 50.165 0)
 		(effects
 			(font
@@
 		)
 	)
-	(text "GPIO PINS ASSIGNMENT (x18)\nIN PROGRESS"
-		(exclude_from_sim no)
-		(at 36.83 199.39 0)
-		(effects
-			(font
-				(size 1.27 1.27)
-			)
-			(justify left bottom)
-		)
-	)
-	(text "RESISTOR SIZING"
-		(exclude_from_sim no)
-		(at 128.905 23.495 0)
-		(effects
-			(font
-				(size 2.54 2.54)
-			)
-			(justify left bottom)
-		)
-	)
 	(text "PINOUT"
 		(exclude_from_sim no)
@@
 		)
 	)
-	(text "IN PROGRESS"
-		(exclude_from_sim no)
-		(at 246.38 50.165 0)
-		(effects
-			(font
-				(size 1.27 1.27)
-			)
-			(justify left bottom)
-		)
-	)
 	(text "VDDA Filtering"
 		(exclude_from_sim no)
@@
 	(symbol
 		(lib_id "power:GND")
-		(at 163.195 76.2 0)
+		(at 163.195 75.565 0)
 		(unit 1)
 		(exclude_from_sim no)
@@
 		(fields_autoplaced yes)
 		(property "Reference" "#PWR024"
-			(at 163.195 82.55 0)
+			(at 163.195 81.915 0)
 			(effects
 				(font
@@
 		)
 		(property "Value" "GND"
-			(at 165.1 77.4699 0)
+			(at 165.1 76.8349 0)
 			(effects
 				(font
@@
 		)
 		(property "Footprint" ""
-			(at 163.195 76.2 0)
+			(at 163.195 75.565 0)
 			(effects
 				(font
@@
 		)
 		(property "Datasheet" ""
-			(at 163.195 76.2 0)
+			(at 163.195 75.565 0)
 			(effects
 				(font
@@
 		)
 		(property "Description" "Power symbol creates a global label with name \"GND\" , ground"
-			(at 163.195 76.2 0)
+			(at 163.195 75.565 0)
 			(effects
 				(font
